File: hardware/kicad/Raindetector/Raindetector.kicad_pcb (KiCad board)
At the start: 2 copper layers, 6 parts, among them J1 I2C, J2 Power_CTRL, J3 Electrode, J4 Heater, Q1 A03400A, U1 ADS1115IDGS

Commit message: PCB layouted for Revision 1
Parts:
- added C1: 100nF, Capacitor_SMD:C_1206_3216Metric_Pad1.33x1.80mm_HandSolder, F.Cu at (92.6, 133.2)
- added R1: 100Ohm, Resistor_SMD:R_1206_3216Metric_Pad1.30x1.75mm_HandSolder, F.Cu at (102.3, 146.8)
- added R2: 100kOhm, Resistor_SMD:R_1206_3216Metric_Pad1.30x1.75mm_HandSolder, F.Cu at (102.3, 142.4)
- added R3: 10kOhm, Resistor_SMD:R_1206_3216Metric_Pad1.30x1.75mm_HandSolder, F.Cu at (102.5, 128.0)
- added R4: 100kOhm, Resistor_SMD:R_1206_3216Metric_Pad1.30x1.75mm_HandSolder, F.Cu at (93.9, 128.0)
- J1: value I2C -> DetektorLeft; footprint Connector_PinSocket_2.54mm:PinSocket_1x04_P2.54mm_Vertical -> Connector_PinHeader_2.54mm:PinHeader_1x08_P2.54mm_Vertical
- J2: value Power_CTRL -> DetektorRight; footprint Connector_PinSocket_2.54mm:PinSocket_1x04_P2.54mm_Vertical -> Connector_PinHeader_2.54mm:PinHeader_1x08_P2.54mm_Vertical
- J3: value Electrode -> HEATER_CTRL; footprint Connector_PinSocket_2.54mm:PinSocket_1x02_P2.54mm_Vertical -> Connector_PinSocket_2.54mm:PinSocket_1x04_P2.54mm_Vertical
- J4: value Heater -> RAIN_SIGNAL; footprint Connector_PinSocket_2.54mm:PinSocket_1x02_P2.54mm_Vertical -> Connector_PinSocket_2.54mm:PinSocket_1x04_P2.54mm_Vertical
- U1: value ADS1115IDGS -> ICM7555xB; footprint Package_SO:TSSOP-10_3x3mm_P0.5mm -> Package_SO:SOIC-8_3.9x4.9mm_P1.27mm
- moved J3 86.7 mm to (84.2, 159.0), turned to 90 degrees
- moved J4 79.5 mm to (105.2, 159.0), turned to 90 degrees
- moved J2 59.2 mm to (109.0, 130.2)
- moved Q1 49.4 mm to (97.0, 144.7), turned to 180 degrees
- moved J1 47.8 mm to (88.0, 130.2)
- moved U1 47.4 mm to (101.2, 133.2)
Connections:
- J1 pad 1: GND -> HEATER_LOW
- J1 pad 2: +3V3 -> HEATER_LOW
- J1 pad 3: SDA -> HEATER_LOW
- J1 pad 4: SCL -> unconnected-(J1-Pin_4-Pad4)
- J2 pad 1: GND -> unconnected-(J2-Pin_1-Pad1)
- J2 pad 2: +5V -> unconnected-(J2-Pin_2-Pad2)
- J2 pad 3: HEATER_EN -> unconnected-(J2-Pin_3-Pad3)
- J2 pad 4: +3V3 -> DETECTOR_A
- J3 pad 1: DETECT_A -> GND
- J3 pad 2: DETECT_B -> +5V
- J4 pad 1: +5V -> GND
- J4 pad 2: HEATER_LOW -> +5V
- U1 pad 1: unconnected-(U1-ADDR-Pad1) -> GND
- U1 pad 2: unconnected-(U1-ALERT/RDY-Pad2) -> DETECTOR_A
- U1 pad 3: GND -> RAIN_FREQ
- U1 pad 4: unconnected-(U1-AIN0-Pad4) -> +3V3
- U1 pad 6: unconnected-(U1-AIN2-Pad6) -> DETECTOR_A
- U1 pad 7: unconnected-(U1-AIN3-Pad7) -> Net-(U1-DISCH)
Routing:
- net +3V3: track 0.00 -> 73.1 mm, vias 0 -> 2
- net +5V: track 0.00 -> 40.6 mm
- net RAIN_FREQ: track 0.00 -> 30.6 mm, vias 0 -> 2
- net DETECTOR_A: track 0.00 -> 23.5 mm
- net HEATER_EN: track 0.00 -> 20.2 mm
- net HEATER_LOW: track 0.00 -> 17.8 mm
- net Net-(U1-DISCH): track 0.00 -> 12.2 mm
- net Net-(Q1-G): track 0.00 -> 7.75 mm
- added copper zone on B.Cu, net GND
- added copper zone on F.Cu, net GND
Other:
- board outline added: 50.1 x 50.1 mm
- board text added: "${TITLE} ${REVISION}"

Commit message: Updated Raindetector - no breaking Changes, Added Assembly-Instructions
Parts:
- Q1: value A03400A -> AO3400A
