File: hardware/kicad/EmptyModule/EmptyModule.kicad_pcb (KiCad board)
At the start: 2 copper layers, 38.4 x 64.6 mm, 2 parts, among them J1 Conn_02x04_Odd_Even, J2 Conn_02x04_Odd_Even

Commit message: Changed EmptyBoard / Usage of DesignBlock
Parts:
- moved J1 1.16 mm to (131.1, 75.2)
- moved J2 1.16 mm to (156.5, 75.2)
Connections:
- J1 pad 2: unconnected-(J1-Pin_2-Pad2) -> 24V
- J1 pad 3: unconnected-(J1-Pin_3-Pad3) -> 3V3
- J1 pad 5: unconnected-(J1-Pin_5-Pad5) -> SDA
- J1 pad 6: unconnected-(J1-Pin_6-Pad6) -> SCL
- J1 pad 8: unconnected-(J1-Pin_8-Pad8) -> GPIO2
- J2 pad 2: unconnected-(J2-Pin_2-Pad2) -> 24V
- J2 pad 3: unconnected-(J2-Pin_3-Pad3) -> 3V3
- J2 pad 5: unconnected-(J2-Pin_5-Pad5) -> SDA
- J2 pad 6: unconnected-(J2-Pin_6-Pad6) -> SCL
- J2 pad 7: unconnected-(J2-Pin_7-Pad7) -> GPIO1
Routing:
- net SCL: track 0.00 -> 26.4 mm
- net 3V3: track 0.00 -> 26.4 mm
- net 24V: track 0.00 -> 26.4 mm
- net GPIO2: track 0.04 -> 26.4 mm
- net SDA: track 0.00 -> 26.4 mm
- net 5V: track 0.00 -> 26.4 mm
- net GPIO1: track 0.04 -> 26.4 mm
