File: hardware/kicad/SolarRadiation/SolarRadiation.kicad_sch (KiCad schematic)
At the start: 16 parts, among them U1 ADS1115IDGS, U2 TMP100

Commit message: Fixed Footprint-Assignments, DesignBlocks
Parts:
- SC1: footprint EnvNode:KXOB25-14X1F -> EnvNode-Footprints:KXOB25-14X1F
Changed lines of the file:
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@@
 			)
 		)
-		(property "Footprint" "EnvNode:KXOB25-14X1F"
+		(property "Footprint" "EnvNode-Footprints:KXOB25-14X1F"
 			(at 37.084 33.02 90)
 			(hide yes)
