File: hardware/kicad/MainBoards/EnvNodeMini/EnvNodeMini.kicad_pcb (KiCad board)
At the start: 2 copper layers, 132 x 70 mm, 20 parts, among them J1 Conn_02x04_Odd_Even, J2 Conn_02x04_Odd_Even, J3 Power, J4 Conn_02x04_Odd_Even, J5 Conn_02x04_Odd_Even, U1 ESP32-DevKitC, U2 24AA025E-OT, U3 TSR_1-2450, U4 TSR_1-2433

Commit message: Changed Footprint for 47uF Elko on EnvNode Mini to SMD
Parts:
- C1: footprint Capacitor_THT:CP_Radial_D6.3mm_P2.50mm -> Capacitor_SMD:CP_Elec_6.3x7.7
Routing:
- net 24V: track 326.9 -> 340.4 mm

Commit message: Changed Value for D1 to B360B-13-F
Parts:
- D1: value STPS3L60S -> B360B-13-F
Changed lines of the file:
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@@
 			)
 		)
-		(property "Value" "STPS3L60S"
+		(property "Value" "B360B-13-F"
 			(at 0 3 0)
 			(layer "F.Fab")
