File: hardware/kicad/MainBoards/EnvNodeMini/EnvNodeMini.kicad_sch (KiCad schematic)
At the start: 16 parts, among them J3 Power, U1 ESP32-DevKitC, U2 24AA025E-OT, U3 TSR_1-2450, U4 TSR_1-2433

Commit message: Changed Footprint for 47uF Elko on EnvNode Mini to SMD
Parts:
- C1: footprint Capacitor_THT:CP_Radial_D6.3mm_P2.50mm -> Capacitor_SMD:CP_Elec_6.3x7.7
Changed lines of the file:
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@@
 		)
 		(instances
-			(project "EnvNodeMIni"
+			(project "EnvNodeMini"
 				(path "/bc65ad1a-48cb-4693-9eab-33a13bb66b0b"
 					(reference "U4")
@@
 		)
 		(instances
-			(project "EnvNodeMIni"
+			(project "EnvNodeMini"
 				(path "/bc65ad1a-48cb-4693-9eab-33a13bb66b0b"
 					(reference "#PWR04")
@@
 		)
 		(instances
-			(project "EnvNodeMIni"
+			(project "EnvNodeMini"
 				(path "/bc65ad1a-48cb-4693-9eab-33a13bb66b0b"
 					(reference "#PWR01")
@@
 		)
 		(instances
-			(project "EnvNodeMIni"
+			(project "EnvNodeMini"
 				(path "/bc65ad1a-48cb-4693-9eab-33a13bb66b0b"
 					(reference "I2C0_1")
@@
 		)
 		(instances
-			(project "EnvNodeMIni"
+			(project "EnvNodeMini"
 				(path "/bc65ad1a-48cb-4693-9eab-33a13bb66b0b"
 					(reference "U3")
@@
 		)
 		(instances
-			(project "EnvNodeMIni"
+			(project "EnvNodeMini"
 				(path "/bc65ad1a-48cb-4693-9eab-33a13bb66b0b"
 					(reference "I2C0_2")
@@
 			)
 		)
-		(property "Footprint" "Capacitor_THT:CP_Radial_D6.3mm_P2.50mm"
+		(property "Footprint" "Capacitor_SMD:CP_Elec_6.3x7.7"
 			(at 93.6752 167.64 0)
 			(hide yes)
@@
 		)
 		(instances
-			(project "EnvNodeMIni"
+			(project "EnvNodeMini"
 				(path "/bc65ad1a-48cb-4693-9eab-33a13bb66b0b"
 					(reference "C1")
@@
 		)
 		(instances
-			(project "EnvNodeMIni"
+			(project "EnvNodeMini"
 				(path "/bc65ad1a-48cb-4693-9eab-33a13bb66b0b"
 					(reference "C2")
@@
 		)
 		(instances
-			(project "EnvNodeMIni"
+			(project "EnvNodeMini"
 				(path "/bc65ad1a-48cb-4693-9eab-33a13bb66b0b"
 					(reference "F1")
@@
 		)
 		(instances
-			(project "EnvNodeMIni"
+			(project "EnvNodeMini"
 				(path "/bc65ad1a-48cb-4693-9eab-33a13bb66b0b"
 					(reference "R1")
@@
 		)
 		(instances
-			(project "EnvNodeMIni"
+			(project "EnvNodeMini"
 				(path "/bc65ad1a-48cb-4693-9eab-33a13bb66b0b"
 					(reference "D2")
@@
 		)
 		(instances
-			(project "EnvNodeMIni"
+			(project "EnvNodeMini"
 				(path "/bc65ad1a-48cb-4693-9eab-33a13bb66b0b"
 					(reference "#PWR08")
@@
 		)
 		(instances
-			(project "EnvNodeMIni"
+			(project "EnvNodeMini"
 				(path "/bc65ad1a-48cb-4693-9eab-33a13bb66b0b"
 					(reference "D1")
@@
 		)
 		(instances
-			(project "EnvNodeMIni"
+			(project "EnvNodeMini"
 				(path "/bc65ad1a-48cb-4693-9eab-33a13bb66b0b"
 					(reference "#PWR03")
@@
 		)
 		(instances
-			(project "EnvNodeMIni"
+			(project "EnvNodeMini"
 				(path "/bc65ad1a-48cb-4693-9eab-33a13bb66b0b"
 					(reference "#PWR06")
@@
 		)
 		(instances
-			(project "EnvNodeMIni"
+			(project "EnvNodeMini"
 				(path "/bc65ad1a-48cb-4693-9eab-33a13bb66b0b"
 					(reference "#PWR05")
@@
 		)
 		(instances
-			(project "EnvNodeMIni"
+			(project "EnvNodeMini"
 				(path "/bc65ad1a-48cb-4693-9eab-33a13bb66b0b"
 					(reference "#PWR09")
@@
 		)
 		(instances
-			(project "EnvNodeMIni"
+			(project "EnvNodeMini"
 				(path "/bc65ad1a-48cb-4693-9eab-33a13bb66b0b"
 					(reference "#FLG01")
@@
 				)
 			)
-			(project "EnvNodeMIni"
+			(project "EnvNodeMini"
 				(path "/bc65ad1a-48cb-4693-9eab-33a13bb66b0b"
 					(reference "J3")
@@
 		)
 		(instances
-			(project "EnvNodeMIni"
+			(project "EnvNodeMini"
 				(path "/bc65ad1a-48cb-4693-9eab-33a13bb66b0b"
 					(reference "JP2")
@@
 		)
 		(instances
-			(project "EnvNodeMIni"
+			(project "EnvNodeMini"
 				(path "/bc65ad1a-48cb-4693-9eab-33a13bb66b0b"
 					(reference "#FLG02")
@@
 		)
 		(instances
-			(project "EnvNodeMIni"
+			(project "EnvNodeMini"
 				(path "/bc65ad1a-48cb-4693-9eab-33a13bb66b0b"
 					(reference "R2")
@@
 		)
 		(instances
-			(project "EnvNodeMIni"
+			(project "EnvNodeMini"
 				(path "/bc65ad1a-48cb-4693-9eab-33a13bb66b0b"
 					(reference "U2")
@@
 		)
 		(instances
-			(project "EnvNodeMIni"
+			(project "EnvNodeMini"
 				(path "/bc65ad1a-48cb-4693-9eab-33a13bb66b0b"
 					(reference "JP1")
@@
 		)
 		(instances
-			(project "EnvNodeMIni"
+			(project "EnvNodeMini"
 				(path "/bc65ad1a-48cb-4693-9eab-33a13bb66b0b"
 					(reference "U1")
@@
 		)
 		(instances
-			(project "EnvNodeMIni"
+			(project "EnvNodeMini"
 				(path "/bc65ad1a-48cb-4693-9eab-33a13bb66b0b"
 					(reference "#PWR02")
@@
 		)
 		(instances
-			(project "EnvNodeMIni"
+			(project "EnvNodeMini"
 				(path "/bc65ad1a-48cb-4693-9eab-33a13bb66b0b"
 					(page "2")
@@
 		)
 		(instances
-			(project "EnvNodeMIni"
+			(project "EnvNodeMini"
 				(path "/bc65ad1a-48cb-4693-9eab-33a13bb66b0b"
 					(page "3")

Commit message: Change Value of D1 to B360B-13-F
Parts:
- D1: value STPS3L60S -> B360B-13-F
Changed lines of the file:
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@@
 			)
 		)
-		(property "Value" "STPS3L60S"
+		(property "Value" "B360B-13-F"
 			(at 71.4375 156.21 0)
 			(show_name no)
