File: hardware/kicad/DesignBlocks/EnvNode_Module_Connector_Daughterboard_SMD/EnvNode_Module_Connector_Daughterboard_SMD.kicad_pcb (KiCad board)
At the start: 2 copper layers, 1 part, among them J1 Conn_02x07_Odd_Even

Commit message: Add EEPROM slot address pin to module interface
Connections:
- J1 pad 3: /GND -> /EEPROM_A0
Changed lines of the file:
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@@
 			(size 1 3.1)
 			(layers "B.Cu" "B.Mask" "B.Paste")
-			(net "/GND")
+			(net "/EEPROM_A0")
 			(pinfunction "Pin_3_3")
 			(pintype "passive")
