File: hardware/kicad/DesignBlocks/EnvNode_Module_Connector_Daughterboard_SMD/EnvNode_Module_Connector_Daughterboard_SMD.kicad_sch (KiCad schematic)
At the start: 1 part, among them J1 Conn_02x07_Odd_Even

Commit message: Add EEPROM slot address pin to module interface
Connections:
- net GND: no longer J1.3 (Pin_3)
- new net EEPROM_A0: J1.3 (Pin_3)
Changed lines of the file:
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@@
 		)
 	)
-	(label "GND"
+	(label "EEPROM_A0"
 		(at 133.35 78.74 180)
 		(effects
