File: hardware/kicad/DesignBlocks/EnvNode_Module_Connector_Daughterboard_THT/EnvNode_Module_Connector_Daughterboard_THT.kicad_pcb (KiCad board)
At the start: 2 copper layers, 1 part, among them J1 Conn_02x07_Odd_Even

Commit message: Add EEPROM slot address pin to module interface
Connections:
- J1 pad 3: /GND -> /EEPROM_A0
Changed lines of the file:
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@@
 		(property ki_fp_filters "Connector*:*_2x??_*")
 		(sheetname "/")
-		(sheetfile "EnvNode_Module_Connector_Daughterboard.kicad_sch")
+		(sheetfile "EnvNode_Module_Connector_Daughterboard_THT.kicad_sch")
 		(units
 			(unit
@@
 			(layers "*.Cu" "*.Mask")
 			(remove_unused_layers no)
-			(net "/GND")
+			(net "/EEPROM_A0")
 			(pinfunction "Pin_3_3")
 			(pintype "passive")
@@
 	)
 	(group ""
-		(lib_id "EnvNodeDesignBlocks:EnvNode_Module_Connector_Daughterboard")
+		(lib_id "EnvNodeDesignBlocks:EnvNode_Module_Connector_Daughterboard_THT")
 		(members "8b7f6c95-da1f-4892-a15d-40780c8e1f28")
 	)
