File: hardware/kicad/Libraries/EnvNodeDesignBlocks.kicad_blocks/EnvNode_Module_Connector_Daughterboard_THT.kicad_block/EnvNode_Module_Connector_Daughterboard_THT.kicad_pcb (KiCad board)
At the start: 2 copper layers, 1 part, among them J1 Conn_02x07_Odd_Even

Commit message: Add EEPROM slot address pin to module interface
Connections:
- J1 pad 3: /GND -> /EEPROM_A0
Changed lines of the file:
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@@
 		(descr "Through hole straight pin header, 2x07, 2.54mm pitch, double rows")
 		(tags "Through hole pin header THT 2x07 2.54mm double row")
+		(property "Reference" "J1"
+			(at 1.27 2.38 0)
+			(layer "B.SilkS")
+			(effects
+				(font
+					(size 1 1)
+					(thickness 0.15)
+				)
+				(justify mirror)
+			)
+		)
+		(property "Value" "Conn_02x07_Odd_Even"
+			(at 1.27 -17.62 0)
+			(layer "B.Fab")
+			(effects
+				(font
+					(size 1 1)
+					(thickness 0.15)
+				)
+				(justify mirror)
+			)
+		)
 		(property "Datasheet" ""
 			(at 0 0 0)
@@
 			)
 		)
-		(property "Reference" "J1"
-			(at 1.27 2.38 0)
-			(layer "B.SilkS")
-			(effects
-				(font
-					(size 1 1)
-					(thickness 0.15)
-				)
-				(justify mirror)
-			)
-		)
-		(property "Value" "Conn_02x07_Odd_Even"
-			(at 1.27 -17.62 0)
-			(layer "B.Fab")
-			(effects
-				(font
-					(size 1 1)
-					(thickness 0.15)
-				)
-				(justify mirror)
-			)
-		)
 		(property ki_fp_filters "Connector*:*_2x??_*")
 		(sheetname "/")
-		(sheetfile "EnvNode_Module_Connector_Daughterboard.kicad_sch")
+		(sheetfile "EnvNode_Module_Connector_Daughterboard_THT.kicad_sch")
 		(attr through_hole)
 		(duplicate_pad_numbers_are_jumpers no)
@@
 			(layers "*.Cu" "*.Mask")
 			(remove_unused_layers no)
-			(net "/GND")
+			(net "/EEPROM_A0")
 			(pinfunction "Pin_3_3")
 			(pintype "passive")
