File: hardware/kicad/Modules/EmptyHalf_SMD/EmptyHalf_SMD.kicad_pcb (KiCad board)
At the start: 2 copper layers, 38 x 32 mm, 2 parts, among them J1 Conn_02x07_Odd_Even

Commit message: Add EEPROM slot address pin to module interface
Connections:
- J1 pad 3: /GND -> /EEPROM_A0
Changed lines of the file:
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@@
 			(size 1 3.1)
 			(layers "B.Cu" "B.Mask" "B.Paste")
-			(net "/GND")
+			(net "/EEPROM_A0")
 			(pinfunction "Pin_3_3")
 			(pintype "passive")
@@
 		)
 	)
-	(group "EnvNode_Module_Connector_Daughterboard_SMD"
-		(lib_id "EnvNodeDesignBlocks:EnvNode_Module_Connector_Daughterboard_SMD")
-		(members "4d689121-2d0a-4948-8561-482f6dc18910")
-	)
 	(embedded_fonts no)
