File: hardware/kicad/Modules/EmptyHalf_THT/EmptyHalf_THT.kicad_pcb (KiCad board)
At the start: 2 copper layers, 38 x 32 mm, 2 parts, among them J1 Conn_02x07_Odd_Even

Commit message: Add EEPROM slot address pin to module interface
Connections:
- J1 pad 3: /GND -> /EEPROM_A0
Changed lines of the file:
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@@
 			(layers "*.Cu" "*.Mask")
 			(remove_unused_layers no)
-			(net "/GND")
+			(net "/EEPROM_A0")
 			(pinfunction "Pin_3_3")
 			(pintype "passive")
-			(zone_connect 2)
 		)
 		(pad "4" thru_hole circle
