File: hardware/kicad/DesignBlocks/ESP32 Core Dual Power ORing/ESP32 Core Dual Power ORing.kicad_pcb (KiCad board)
At the start: 2 copper layers, 7 parts, among them U1 ESP32-DevKitC, U3 24LC32

Commit message: Refine ESP32 core EEPROM layout
Parts:
- moved C3 5.84 mm to (229.0, 72.9), turned to 180 degrees
Routing:
- net GND: track 5.47 -> 0.00 mm
- net +3V3_SYS: track 22.7 -> 24.5 mm
Changed lines of the file:
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@@
+		)
+	)
+	(footprint "Capacitor_SMD:C_1206_3216Metric_Pad1.33x1.80mm_HandSolder"
+		(layer "F.Cu")
+		(at 229.04 72.94 180)
+		(descr "Capacitor SMD 1206 (3216 Metric), square (rectangular) end terminal, IPC-7351 nominal with elongated pad for handsoldering. (Body size source: IPC-SM-782 page 76, https://www.pcb-3d.com/wordpress/wp-content/uploads/ipc-sm-782a_amendment_1_and_2.pdf)")
+		(tags "capacitor handsolder")
+		(property "Reference" "C3"
+			(at 3.65 -0.01 180)
+			(layer "F.SilkS")
+			(effects
+				(font
+					(size 1 1)
+					(thickness 0.15)
+				)
+			)
+		)
+		(property "Value" "100nF"
+			(at 0 1.85 90)
+			(layer "F.Fab")
+			(effects
+				(font
+					(size 1 1)
+					(thickness 0.15)
+				)
+			)
+		)
+		(property "Datasheet" ""
+			(at 0 0 90)
+			(layer "F.Fab")
+			(hide yes)
+			(effects
+				(font
+					(size 1.27 1.27)
+				)
+			)
+		)
+		(property "Description" "Unpolarized capacitor"
+			(at 0 0 90)
+			(layer "F.Fab")
+			(hide yes)
+			(effects
+				(font
+					(size 1.27 1.27)
+				)
+			)
+		)
+		(property "KiLib_Generator" "SMD_2terminal_chip_molded"
+			(at 0 0 90)
+			(layer "F.SilkS")
+			(hide yes)
+			(effects
+				(font
+					(size 1 1)
+					(thickness 0.15)
+				)
+			)
+		)
+		(property ki_fp_filters "C_*")
+		(sheetname "/")
+		(sheetfile "ESP32 Core Dual Power ORing.kicad_sch")
+		(units
+			(unit
+				(name "A")
+				(pins "1" "2")
+			)
+		)
+		(attr smd)
+		(duplicate_pad_numbers_are_jumpers no)
+		(fp_line
+			(start -0.711252 0.91)
+			(end 0.711252 0.91)
+			(stroke
+				(width 0.12)
+				(type solid)
+			)
+			(layer "F.SilkS")
+		)
+		(fp_line
+			(start -0.711252 -0.91)
+			(end 0.711252 -0.91)
+			(stroke
+				(width 0.12)
+				(type solid)
+			)
+			(layer "F.SilkS")
+		)
+		(fp_rect
+			(start -2.48 -1.15)
+			(end 2.48 1.15)
+			(stroke
+				(width 0.05)
+				(type solid)
+			)
+			(fill no)
+			(layer "F.CrtYd")
+		)
+		(fp_rect
+			(start -1.6 -0.8)
+			(end 1.6 0.8)
+			(stroke
+				(width 0.1)
+				(type solid)
+			)
+			(fill no)
+			(layer "F.Fab")
+		)
+		(fp_text user "${REFERENCE}"
+			(at 0 0 90)
+			(layer "F.Fab")
+			(effects
+				(font
+					(size 0.8 0.8)
+					(thickness 0.12)
+				)
+			)
+		)
+		(pad "1" smd roundrect
+			(at -1.5625 0 270)
+			(size 1.325 1.8)
+			(layers "F.Cu" "F.Mask" "F.Paste")
+			(roundrect_rratio 0.188679)
+			(net "+3V3_SYS")
+			(pintype "passive")
+		)
+		(pad "2" smd roundrect
+			(at 1.5625 0 270)
+			(size 1.325 1.8)
+			(layers "F.Cu" "F.Mask" "F.Paste")
+			(roundrect_rratio 0.188679)
+			(net "GND")
+			(pintype "passive")
+		)
+		(embedded_fonts no)
+		(model "${KICAD10_3DMODEL_DIR}/Capacitor_SMD.3dshapes/C_1206_3216Metric.step"
+			(offset
+				(xyz 0 0 0)
+			)
+			(scale
+				(xyz 1 1 1)
+			)
+			(rotate
+				(xyz 0 0 0)
+			)
 		)
 	)
 	(footprint "Package_SO:SOIC-8_3.9x4.9mm_P1.27mm"
+		(locked yes)
 		(layer "F.Cu")
 		(at 229.04 78.1875)
@@
 	)
 	(segment
+		(start 231.515 76.2825)
+		(end 230.6025 75.37)
+		(width 0.2)
+		(layer "F.Cu")
+		(net "+3V3_SYS")
+	)
+	(segment
 		(start 187.036447 69.91)
 		(end 187.652706 69.293741)
@@
 	)
 	(segment
+		(start 230.6025 75.37)
+		(end 230.6025 72.94)
+		(width 0.2)
+		(layer "F.Cu")
+		(net "+3V3_SYS")
+	)
+	(segment
 		(start 196.03 65.81)
 		(end 187.742706 65.81)
@@
 	)
 	(segment
-		(start 228.76 75.11)
-		(end 228.023741 74.373741)
+		(start 229.7575 80.0925)
+		(end 227.856259 81.993741)
+		(width 0.2)
+		(layer "F.Cu")
+		(net "I2C0_SDA")
+	)
+	(segment
+		(start 231.515 80.0925)
+		(end 229.7575 80.0925)
+		(width 0.2)
+		(layer "F.Cu")
+		(net "I2C0_SDA")
+	)
+	(segment
+		(start 227.856259 81.993741)
+		(end 222.352706 81.993741)
+		(width 0.2)
+		(layer "F.Cu")
+		(net "I2C0_SDA")
+	)
+	(segment
+		(start 228.043741 74.373741)
+		(end 228.76 75.09)
 		(width 0.2)
 		(layer "F.Cu")
@@
 	)
 	(segment
-		(start 228.023741 74.373741)
-		(end 222.352706 74.373741)
+		(start 222.352706 74.373741)
+		(end 228.043741 74.373741)
 		(width 0.2)
 		(layer "F.Cu")
@@
 	)
 	(segment
-		(start 228.76 77.88)
-		(end 228.76 75.11)
+		(start 228.76 75.09)
+		(end 228.76 77.88)
 		(width 0.2)
 		(layer "F.Cu")
 		(net "I2C0_SCL")
 	)
-	(segment
-		(start 229.7575 80.0925)
-		(end 227.856259 81.993741)
-		(width 0.2)
-		(layer "F.Cu")
-		(net "I2C0_SDA")
-	)
-	(segment
-		(start 231.515 80.0925)
-		(end 229.7575 80.0925)
-		(width 0.2)
-		(layer "F.Cu")
-		(net "I2C0_SDA")
-	)
-	(segment
-		(start 227.856259 81.993741)
-		(end 222.352706 81.993741)
-		(width 0.2)
-		(layer "F.Cu")
-		(net "I2C0_SDA")
-	)
-	(group ""
-		(lib_id "EnvNodeDesignBlocks:ESP32 Core Dual Power ORing")
-		(members "03044a93-e572-405e-8451-31c5de8456a0" "22fa1f00-6f61-49c7-bd04-cb7d98db8aa7"
-			"2db9e568-1b3e-44e5-a1bc-52eb6443b44e" "2f944301-0968-47ac-8858-10bc613d2dc5"
-			"3a6a89d8-3f3e-4031-a595-8703f545c961" "41f533f0-8bda-4c95-b0a6-b3298074d7fb"
-			"4964c117-c18c-48b6-8f7d-319d1ea7c878" "5b1428eb-0bd1-4caa-aa61-44494c087c59"
-			"64417791-c4ca-4af7-8bf9-aa0928513777" "66cce79a-4bfc-4913-ad00-f6bdbe0b138c"
-			"70e0759d-a42e-4a1e-934c-eaa5e8d77eb1" "7884c9de-41bc-497b-8f57-36d84f7ba39c"
-			"87f8975e-2d1b-4d0d-9473-ffbffbb1b254" "906605b4-3e52-4cd7-9935-d4bd84fe79fa"
-			"952dbd5a-a8b5-4513-a073-2b46ea2e8326" "a2d0ca58-da91-46c1-9683-954b9b6b19bf"
-			"b297a62e-a5ec-4f9a-bd4b-e7bc591aeca2" "be3278c6-d81c-4f3c-a94d-993c873b6da6"
-			"d339221a-1791-45fe-819e-5d12eb834057" "d6463d19-86c1-4027-9fb8-239c62094e05"
-			"dc186229-dbf9-45dd-a908-af95ce3ea041" "de3b910c-4d78-4ed4-b00f-2dc802278c13"
-			"ecb6d293-0203-4a45-a40f-c0339998514c"
-		)
-	)
 	(embedded_fonts no)
-	(footprint "Capacitor_SMD:C_1206_3216Metric_Pad1.33x1.80mm_HandSolder"
-		(layer "F.Cu")
-		(at 234.5 75)
-		(descr "Capacitor SMD 1206 (3216 Metric), square (rectangular) end terminal, IPC-7351 nominal with elongated pad for handsoldering. (Body size source: IPC-SM-782 page 76, https://www.pcb-3d.com/wordpress/wp-content/uploads/ipc-sm-782a_amendment_1_and_2.pdf)")
-		(tags "capacitor handsolder")
-		(property "Reference" "C3"
-			(at 0 -1.85 90)
-			(layer "F.SilkS")
-			(effects
-				(font
-					(size 1 1)
-					(thickness 0.15)
-				)
-			)
-		)
-		(property "Value" "100nF"
-			(at 0 1.85 90)
-			(layer "F.Fab")
-			(effects
-				(font
-					(size 1 1)
-					(thickness 0.15)
-				)
-			)
-		)
-		(property "Datasheet" ""
-			(at 0 0 90)
-			(layer "F.Fab")
-			(hide yes)
-			(effects
-				(font
-					(size 1.27 1.27)
-				)
-			)
-		)
-		(property "Description" "Unpolarized capacitor"
-			(at 0 0 90)
-			(layer "F.Fab")
-			(hide yes)
-			(effects
-				(font
-					(size 1.27 1.27)
-				)
-			)
-		)
-		(property "KiLib_Generator" "SMD_2terminal_chip_molded"
-			(at 0 0 90)
-			(layer "F.SilkS")
-			(hide yes)
-			(effects
-				(font
-					(size 1 1)
-					(thickness 0.15)
-				)
-			)
-		)
-		(property ki_fp_filters "C_*")
-		(sheetname "/")
-		(sheetfile "ESP32 Core Dual Power ORing.kicad_sch")
-		(units
-			(unit
-				(name "A")
-				(pins "1" "2")
-			)
-		)
-		(attr smd)
-		(duplicate_pad_numbers_are_jumpers no)
-		(fp_line
-			(start -0.711252 -0.91)
-			(end 0.711252 -0.91)
-			(stroke
-				(width 0.12)
-				(type solid)
-			)
-			(layer "F.SilkS")
-		)
-		(fp_line
-			(start -0.711252 0.91)
-			(end 0.711252 0.91)
-			(stroke
-				(width 0.12)
-				(type solid)
-			)
-			(layer "F.SilkS")
-		)
-		(fp_rect
-			(start -2.48 -1.15)
-			(end 2.48 1.15)
-			(stroke
-				(width 0.05)
-				(type solid)
-			)
-			(fill no)
-			(layer "F.CrtYd")
-		)
-		(fp_rect
-			(start -1.6 -0.8)
-			(end 1.6 0.8)
-			(stroke
-				(width 0.1)
-				(type solid)
-			)
-			(fill no)
-			(layer "F.Fab")
-		)
-		(fp_text user "${REFERENCE}"
-			(at 0 0 90)
-			(layer "F.Fab")
-			(effects
-				(font
-					(size 0.8 0.8)
-					(thickness 0.12)
-				)
-			)
-		)
-		(pad "1" smd roundrect
-			(at -1.5625 0 90)
-			(size 1.325 1.8)
-			(layers "F.Cu" "F.Mask" "F.Paste")
-			(roundrect_rratio 0.188679)
-			(net "+3V3_SYS")
-			(pintype "passive")
-		)
-		(pad "2" smd roundrect
-			(at 1.5625 0 90)
-			(size 1.325 1.8)
-			(layers "F.Cu" "F.Mask" "F.Paste")
-			(roundrect_rratio 0.188679)
-			(net "GND")
-			(pintype "passive")
-		)
-		(embedded_fonts no)
-		(model "${KICAD10_3DMODEL_DIR}/Capacitor_SMD.3dshapes/C_1206_3216Metric.step"
-			(offset
-				(xyz 0 0 0)
-			)
-			(scale
-				(xyz 1 1 1)
-			)
-			(rotate
-				(xyz 0 0 0)
-			)
-		)
-	)
-	(segment
-		(start 231.515 76.2825)
-		(end 232.9375 75)
-		(width 0.2)
-		(layer "F.Cu")
-		(net "+3V3_SYS")
-	)
-	(segment
-		(start 236.0625 75)
-		(end 233 77.5525)
-		(width 0.2)
-		(layer "F.Cu")
-		(net "GND")
-	)
-	(segment
-		(start 233 77.5525)
-		(end 231.515 77.5525)
-		(width 0.2)
-		(layer "F.Cu")
-		(net "GND")
-	)
 )
