File: hardware/kicad/DesignBlocks/ORing Power/ORing Power.kicad_sch (KiCad schematic)
At the start: 13 parts, among them J1 Conn_01x02_Pin, J3 USB_C_Receptacle_PowerOnly_6P, U1 LM3940IMP-3.3/NOPB, U2 ORingPower_Module

Commit message: fix(hardware): use SMD JST-PH on ORing power module
Parts:
- J1: footprint Connector_JST:JST_PH_B2B-PH-K_1x02_P2.00mm_Vertical -> Connector_JST:JST_PH_B2B-PH-SM4-TB_1x02-1MP_P2.00mm_Vertical
Changed lines of the file:
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@@
 			)
 		)
-		(property "Footprint" "Connector_JST:JST_PH_B2B-PH-K_1x02_P2.00mm_Vertical"
+		(property "Footprint" "Connector_JST:JST_PH_B2B-PH-SM4-TB_1x02-1MP_P2.00mm_Vertical"
 			(at 58.42 99.06 0)
 			(hide yes)
