File: hardware/kicad/DesignBlocks/BOX4U-5U210900/BOX4U-5U210900.kicad_pcb (KiCad board)
At the start: 2 copper layers, 130 x 68 mm, 4 parts

Commit message: feat(hardware): complete BOX4U geometry design block
Parts:
- H1, H2, H3, H4: footprint MountingHole_4.5mm_SelfTapping_4mm -> EnvNode-Footprints:MountingHole_4.5mm_SelfTapping_4mm
Changed lines of the file:
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@@
     (allow_soldermask_bridges_in_footprints no)
   )
-  (footprint "MountingHole_4.5mm_SelfTapping_4mm"
+  (footprint "EnvNode-Footprints:MountingHole_4.5mm_SelfTapping_4mm"
     (layer "F.Cu")
     (at 39.25 71)
     (property "Reference" "H1" (at 0 -5.5 0) (layer "F.SilkS") (hide yes) (effects (font (size 1 1) (thickness 0.15))))
     (property "Value" "Self-tapping 4 mm / NPTH 4.5 mm" (at 0 5.5 0) (layer "F.Fab") (hide yes) (effects (font (size 1 1) (thickness 0.15))))
+    (sheetname "/")
+    (sheetfile "BOX4U-5U210900.kicad_sch")
     (fp_circle (center 0 0) (end 4.5 0) (stroke (width 0.25) (type solid)) (fill none) (layer "F.CrtYd"))
     (pad "" np_thru_hole circle (at 0 0) (size 4.5 4.5) (drill 4.5) (layers "*.Cu" "*.Mask") (clearance 2.25))
   )
-  (footprint "MountingHole_4.5mm_SelfTapping_4mm"
+  (footprint "EnvNode-Footprints:MountingHole_4.5mm_SelfTapping_4mm"
     (layer "F.Cu")
     (at 160.75 71)
     (property "Reference" "H2" (at 0 -5.5 0) (layer "F.SilkS") (hide yes) (effects (font (size 1 1) (thickness 0.15))))
     (property "Value" "Self-tapping 4 mm / NPTH 4.5 mm" (at 0 5.5 0) (layer "F.Fab") (hide yes) (effects (font (size 1 1) (thickness 0.15))))
+    (sheetname "/")
+    (sheetfile "BOX4U-5U210900.kicad_sch")
     (fp_circle (center 0 0) (end 4.5 0) (stroke (width 0.25) (type solid)) (fill none) (layer "F.CrtYd"))
     (pad "" np_thru_hole circle (at 0 0) (size 4.5 4.5) (drill 4.5) (layers "*.Cu" "*.Mask") (clearance 2.25))
   )
-  (footprint "MountingHole_4.5mm_SelfTapping_4mm"
+  (footprint "EnvNode-Footprints:MountingHole_4.5mm_SelfTapping_4mm"
     (layer "F.Cu")
     (at 160.75 129)
     (property "Reference" "H3" (at 0 -5.5 0) (layer "F.SilkS") (hide yes) (effects (font (size 1 1) (thickness 0.15))))
     (property "Value" "Self-tapping 4 mm / NPTH 4.5 mm" (at 0 5.5 0) (layer "F.Fab") (hide yes) (effects (font (size 1 1) (thickness 0.15))))
+    (sheetname "/")
+    (sheetfile "BOX4U-5U210900.kicad_sch")
     (fp_circle (center 0 0) (end 4.5 0) (stroke (width 0.25) (type solid)) (fill none) (layer "F.CrtYd"))
     (pad "" np_thru_hole circle (at 0 0) (size 4.5 4.5) (drill 4.5) (layers "*.Cu" "*.Mask") (clearance 2.25))
   )
-  (footprint "MountingHole_4.5mm_SelfTapping_4mm"
+  (footprint "EnvNode-Footprints:MountingHole_4.5mm_SelfTapping_4mm"
     (layer "F.Cu")
     (at 39.25 129)
     (property "Reference" "H4" (at 0 -5.5 0) (layer "F.SilkS") (hide yes) (effects (font (size 1 1) (thickness 0.15))))
     (property "Value" "Self-tapping 4 mm / NPTH 4.5 mm" (at 0 5.5 0) (layer "F.Fab") (hide yes) (effects (font (size 1 1) (thickness 0.15))))
+    (sheetname "/")
+    (sheetfile "BOX4U-5U210900.kicad_sch")
     (fp_circle (center 0 0) (end 4.5 0) (stroke (width 0.25) (type solid)) (fill none) (layer "F.CrtYd"))
     (pad "" np_thru_hole circle (at 0 0) (size 4.5 4.5) (drill 4.5) (layers "*.Cu" "*.Mask") (clearance 2.25))

Commit message: feat(hardware): complete EnvNode Mini revision 0.6
Parts:
- H1, H2, H3, H4: value Self-tapping 4 mm / NPTH 4.5 mm -> MountingHole
