File: hardware/kicad/DesignBlocks/BOX4U-5U210900/BOX4U-5U210900.kicad_sch (KiCad schematic)
At the start: 0 parts

Commit message: feat(hardware): complete BOX4U geometry design block
Parts:
- added H1, H2, H3, H4: MountingHole, EnvNode-Footprints:MountingHole_4.5mm_SelfTapping_4mm, symbol Mechanical:MountingHole
Changed lines of the file:
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@@
   (generator_version "9.0")
   (paper "A4")
+  (symbol
+    (lib_id "Mechanical:MountingHole") (at 76.2 63.5 0) (unit 1) (body_style 1)
+    (exclude_from_sim no) (in_bom no) (on_board yes) (in_pos_files no) (dnp no) (fields_autoplaced yes)
+    (property "Reference" "H1" (at 78.74 62.2299 0) (show_name no) (do_not_autoplace no) (effects (font (size 1.27 1.27)) (justify left)))
+    (property "Value" "MountingHole" (at 78.74 64.7699 0) (show_name no) (do_not_autoplace no) (effects (font (size 1.27 1.27)) (justify left)))
+    (property "Footprint" "EnvNode-Footprints:MountingHole_4.5mm_SelfTapping_4mm" (at 76.2 63.5 0) (hide yes) (show_name no) (do_not_autoplace no) (effects (font (size 1.27 1.27))))
+    (property "Datasheet" "" (at 76.2 63.5 0) (hide yes) (show_name no) (do_not_autoplace no) (effects (font (size 1.27 1.27))))
+    (property "Description" "BOX4U mounting hole: NPTH 4.5 mm for 4 mm self-tapping screw" (at 76.2 63.5 0) (hide yes) (show_name no) (do_not_autoplace no) (effects (font (size 1.27 1.27))))
+    (instances (project "BOX4U-5U210900" (path "/23fc823c-9a98-4c93-a80e-354672461955" (reference "H1") (unit 1))))
+  )
+  (symbol
+    (lib_id "Mechanical:MountingHole") (at 127 63.5 0) (unit 1) (body_style 1)
+    (exclude_from_sim no) (in_bom no) (on_board yes) (in_pos_files no) (dnp no) (fields_autoplaced yes)
+    (property "Reference" "H2" (at 129.54 62.2299 0) (show_name no) (do_not_autoplace no) (effects (font (size 1.27 1.27)) (justify left)))
+    (property "Value" "MountingHole" (at 129.54 64.7699 0) (show_name no) (do_not_autoplace no) (effects (font (size 1.27 1.27)) (justify left)))
+    (property "Footprint" "EnvNode-Footprints:MountingHole_4.5mm_SelfTapping_4mm" (at 127 63.5 0) (hide yes) (show_name no) (do_not_autoplace no) (effects (font (size 1.27 1.27))))
+    (property "Datasheet" "" (at 127 63.5 0) (hide yes) (show_name no) (do_not_autoplace no) (effects (font (size 1.27 1.27))))
+    (property "Description" "BOX4U mounting hole: NPTH 4.5 mm for 4 mm self-tapping screw" (at 127 63.5 0) (hide yes) (show_name no) (do_not_autoplace no) (effects (font (size 1.27 1.27))))
+    (instances (project "BOX4U-5U210900" (path "/23fc823c-9a98-4c93-a80e-354672461955" (reference "H2") (unit 1))))
+  )
+  (symbol
+    (lib_id "Mechanical:MountingHole") (at 127 88.9 0) (unit 1) (body_style 1)
+    (exclude_from_sim no) (in_bom no) (on_board yes) (in_pos_files no) (dnp no) (fields_autoplaced yes)
+    (property "Reference" "H3" (at 129.54 87.6299 0) (show_name no) (do_not_autoplace no) (effects (font (size 1.27 1.27)) (justify left)))
+    (property "Value" "MountingHole" (at 129.54 90.1699 0) (show_name no) (do_not_autoplace no) (effects (font (size 1.27 1.27)) (justify left)))
+    (property "Footprint" "EnvNode-Footprints:MountingHole_4.5mm_SelfTapping_4mm" (at 127 88.9 0) (hide yes) (show_name no) (do_not_autoplace no) (effects (font (size 1.27 1.27))))
+    (property "Datasheet" "" (at 127 88.9 0) (hide yes) (show_name no) (do_not_autoplace no) (effects (font (size 1.27 1.27))))
+    (property "Description" "BOX4U mounting hole: NPTH 4.5 mm for 4 mm self-tapping screw" (at 127 88.9 0) (hide yes) (show_name no) (do_not_autoplace no) (effects (font (size 1.27 1.27))))
+    (instances (project "BOX4U-5U210900" (path "/23fc823c-9a98-4c93-a80e-354672461955" (reference "H3") (unit 1))))
+  )
+  (symbol
+    (lib_id "Mechanical:MountingHole") (at 76.2 88.9 0) (unit 1) (body_style 1)
+    (exclude_from_sim no) (in_bom no) (on_board yes) (in_pos_files no) (dnp no) (fields_autoplaced yes)
+    (property "Reference" "H4" (at 78.74 87.6299 0) (show_name no) (do_not_autoplace no) (effects (font (size 1.27 1.27)) (justify left)))
+    (property "Value" "MountingHole" (at 78.74 90.1699 0) (show_name no) (do_not_autoplace no) (effects (font (size 1.27 1.27)) (justify left)))
+    (property "Footprint" "EnvNode-Footprints:MountingHole_4.5mm_SelfTapping_4mm" (at 76.2 88.9 0) (hide yes) (show_name no) (do_not_autoplace no) (effects (font (size 1.27 1.27))))
+    (property "Datasheet" "" (at 76.2 88.9 0) (hide yes) (show_name no) (do_not_autoplace no) (effects (font (size 1.27 1.27))))
+    (property "Description" "BOX4U mounting hole: NPTH 4.5 mm for 4 mm self-tapping screw" (at 76.2 88.9 0) (hide yes) (show_name no) (do_not_autoplace no) (effects (font (size 1.27 1.27))))
+    (instances (project "BOX4U-5U210900" (path "/23fc823c-9a98-4c93-a80e-354672461955" (reference "H4") (unit 1))))
+  )
   (sheet_instances
     (path "/" (page "1"))
   )
+  (embedded_fonts no)
 )
