File: hardware/kicad/Libraries/EnvNodeDesignBlocks.kicad_blocks/BOX4U-5U210900.kicad_block/BOX4U-5U210900.kicad_pcb (KiCad board)
At the start: 2 copper layers, 130 x 68 mm, 4 parts

Commit message: feat(hardware): complete EnvNode Mini revision 0.6
Parts:
- H1, H2, H3, H4: value Self-tapping 4 mm / NPTH 4.5 mm -> MountingHole
