File: hardware/kicad/MainBoards/Weatherstation/gpio.kicad_sch (KiCad schematic)
At the start: 10 parts

Commit message: hardware(weather): swap slot GPIO4 with GPIO33 for analog input
Parts:
- renumbered GPIO33 to GPIO4
Connections:
- net GPIO33 renamed GPIO4
Changed lines of the file:
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@@
 		)
 	)
-	(hierarchical_label "GPIO33"
+	(hierarchical_label "GPIO4"
 		(shape input)
 		(at 260.35 102.87 270)
@@
 		(dnp no)
 		(fields_autoplaced yes)
-		(property "Reference" "GPIO33"
+		(property "Reference" "GPIO4"
 			(at 261.62 92.71 90)
 			(show_name no)
@@
 			(project "Weatherstation"
 				(path "/bb35dba2-ff1a-441b-885c-8dff8d3b7ea1/52d09e00-3392-4a75-97d4-fe6c18a37b92"
-					(reference "GPIO33")
-					(unit 1)
-				)
+					(reference "GPIO4")
+					(unit 1)
+				)
