File: hardware/kicad/Libraries/EnvNodeDesignBlocks.kicad_blocks/EnvNode_Module_Connector_MainBoard.kicad_block/EnvNode_Module_Connector_MainBoard.kicad_pcb (KiCad board)
At the start: 2 copper layers, 3 parts, among them J1 Conn_02x07_Odd_Even

Commit message: Align mainboard module connector geometry
Parts:
- moved J1 30.3 mm to (119.4, 51.2)
- moved H2 30.3 mm to (127.0, 105.2)
- moved H1 30.3 mm to (127.0, 73.2)
Changed lines of the file:
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@@
 	(footprint "MountingHole:MountingHole_2.7mm_M2.5"
 		(layer "F.Cu")
-		(at 113.08 78.308)
+		(at 127.05 105.156)
 		(descr "Mounting Hole 2.7mm, M2.5, no annular, generated by kicad-footprint-generator mountinghole.py")
 		(tags "mountinghole M2.5")
@@
 	(footprint "Connector_PinSocket_2.54mm:PinSocket_2x07_P2.54mm_Vertical"
 		(layer "F.Cu")
-		(at 105.46 24.38 90)
+		(at 119.43 51.236 90)
 		(descr "Through hole straight socket strip, 2x07, 2.54mm pitch, double rows (from Kicad 4.0.7), script generated")
 		(tags "Through hole socket strip THT 2x07 2.54mm double row")
@@
 	(footprint "MountingHole:MountingHole_2.7mm_M2.5"
 		(layer "F.Cu")
-		(at 113.08 46.318)
+		(at 127.05 73.156)
 		(descr "Mounting Hole 2.7mm, M2.5, no annular, generated by kicad-footprint-generator mountinghole.py")
 		(tags "mountinghole M2.5")
@@
 	)
 	(gr_rect
-		(start 94.08 19.308)
-		(end 132.08 83.308)
+		(start 108.05 46.156)
+		(end 146.05 110.156)
 		(stroke
 			(width 0.1)

Commit message: Add EEPROM slot address pin to module interface
Connections:
- J1 pad 3: /GND -> /EEPROM_A0
Changed lines of the file:
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@@
 			(layers "*.Cu" "*.Mask")
 			(remove_unused_layers no)
-			(net "/GND")
+			(net "/EEPROM_A0")
 			(pinfunction "Pin_3_3")
 			(pintype "passive")
