File: hardware/kicad/Sensors/SCT013Head/SCT013Head.kicad_pcb (KiCad board)
At the start: 2 copper layers, 20.8 x 14 mm, 7 parts, among them J1 Conn_01x05_Pin

Commit message: hardware(sct013): add input attenuator and update kit parts
Parts:
- added R4: 10k, Resistor_SMD:R_1206_3216Metric_Pad1.30x1.75mm_HandSolder, B.Cu at (94.5, 63.8)
- ADC1: footprint Connector_PinSocket_2.54mm:PinSocket_1x04_P2.54mm_Vertical -> Connector_PinHeader_2.54mm:PinHeader_1x04_P2.54mm_Vertical
- R1: value 1k -> 10k
- moved R1 6.96 mm to (89.2, 59.2)
- moved C1 3.26 mm to (91.9, 63.8)
Routing:
- net Net-(J1-Pin_3): track 11.8 -> 5.01 mm
- net ADC: track 12.8 -> 18.4 mm
