File: hardware/kicad/MainBoards/Test-Provisioning/INL.kicad_sch (KiCad schematic)
At the start: 7 parts, among them J4 ESP32_DevKitC_TestPlug, U4 CD74HC4067M, U5 CD74HC4067M, U6 CD74HC4067M

Commit message: Preserve final monolithic fixture state before retiring project
Parts:
- added J7: Conn_01x02_Socket, Connector_PinHeader_2.54mm:PinHeader_1x02_P2.54mm_Vertical, symbol Connector:Conn_01x02_Socket
Connections:
- net MB_GND: now reaches U6.17 (I14)
- net MB_GND: now also J7.2 (Pin_2)
- net MB_3V3_SYS: now reaches U6.18 (I13)
- net MB_3V3_SYS: now also J7.1 (Pin_1)
- no-connect marks 10 -> 8
Changed lines of the file:
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@@
-	)
-	(no_connect
-		(at 243.84 114.3)
 	)
 	(no_connect
 		(at 243.84 116.84)
-	)
-	(no_connect
-		(at 243.84 111.76)
 	)
 	(no_connect
@@
 		)
 	)
+	(label "MB_GND"
+		(at 243.84 114.3 0)
+		(effects
+			(font
+				(size 1.27 1.27)
+			)
+			(justify left bottom)
+		)
+	)
 	(label "L11"
 		(at 43.18 102.87 180)
@@
 		)
 	)
+	(label "MB_GND"
+		(at 257.81 124.46 90)
+		(effects
+			(font
+				(size 1.27 1.27)
+			)
+			(justify left bottom)
+		)
+	)
 	(label "L03"
 		(at 134.62 91.44 0)
@@
 		)
 	)
+	(label "MB_3V3_SYS"
+		(at 243.84 111.76 0)
+		(effects
+			(font
+				(size 1.27 1.27)
+			)
+			(justify left bottom)
+		)
+	)
 	(label "R15"
 		(at 243.84 99.06 0)
@@
 	(label "R06"
 		(at 73.66 90.17 0)
+		(effects
+			(font
+				(size 1.27 1.27)
+			)
+			(justify left bottom)
+		)
+	)
+	(label "MB_3V3_SYS"
+		(at 260.35 124.46 90)
 		(effects
 			(font
@@
 					(unit 1)
 				)
+			)
+		)
+	)
+	(symbol
+		(lib_id "Connector:Conn_01x02_Socket")
+		(at 260.35 129.54 270)
+		(unit 1)
+		(body_style 1)
+		(exclude_from_sim no)
+		(in_bom yes)
+		(on_board yes)
+		(in_pos_files yes)
+		(dnp yes)
+		(fields_autoplaced yes)
+		(property "Reference" "J7"
+			(at 261.62 127.6349 90)
+			(show_name no)
+			(do_not_autoplace no)
+			(effects
+				(font
+					(size 1.27 1.27)
+				)
+				(justify left)
+			)
+		)
+		(property "Value" "Conn_01x02_Socket"
+			(at 261.62 130.1749 90)
+			(show_name no)
+			(do_not_autoplace no)
+			(effects
+				(font
+					(size 1.27 1.27)
+				)
+				(justify left)
+			)
+		)
+		(property "Footprint" "Connector_PinHeader_2.54mm:PinHeader_1x02_P2.54mm_Vertical"
+			(at 260.35 129.54 0)
+			(hide yes)
+			(show_name no)
+			(do_not_autoplace no)
+			(effects
+				(font
+					(size 1.27 1.27)
+				)
+			)
+		)
+		(property "Datasheet" ""
+			(at 260.35 129.54 0)
+			(hide yes)
+			(show_name no)
+			(do_not_autoplace no)
+			(effects
+				(font
+					(size 1.27 1.27)
+				)
+			)
+		)
+		(property "Description" "Generic connector, single row, 01x02, script generated"
+			(at 260.35 129.54 0)
+			(hide yes)
+			(show_name no)
+			(do_not_autoplace no)
+			(effects
+				(font
+					(size 1.27 1.27)
+				)
+			)
+		)
+		(pin "1"
+		)
+		(pin "2"
+		)
+		(instances
+			(project "Test-Provisioning"
+				(path "/8e8be5f8-638f-4444-a554-6e489d9dce34/5d9b3800-6c59-4395-90ab-0ced0ede5c92"
+					(reference "J7")
+					(unit 1)
+				)
