File: hardware/kicad/MainBoards/Input-Adapter/INL.kicad_sch (KiCad schematic)
At the start: 8 parts, among them J4 ESP32_DevKitC_TestPlug, J7 Conn_01x02_Socket, U4 CD74HC4067M, U5 CD74HC4067M, U6 CD74HC4067M

Commit message: Document split test fixture projects and retire monolithic board
Connections:
- net IN_EN1 renamed h_EN1
- net IN_EN2 renamed h_EN2
- net IN_EN3 renamed h_EN3
- net IN_S0 renamed h_S0
- net IN_S1 renamed h_S1
- net IN_S2 renamed h_S2
- net IN_S3 renamed h_S3
Changed lines of the file:
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@@
 		)
 	)
-	(hierarchical_label "IN_S0"
+	(hierarchical_label "h_S0"
 		(shape input)
 		(at 109.22 93.98 180)
@@
 		)
 	)
-	(hierarchical_label "IN_S1"
+	(hierarchical_label "h_S1"
 		(shape input)
 		(at 218.44 96.52 180)
@@
 		)
 	)
-	(hierarchical_label "IN_EN3"
+	(hierarchical_label "h_EN3"
 		(shape input)
 		(at 218.44 111.76 180)
@@
 		)
 	)
-	(hierarchical_label "IN_S3"
+	(hierarchical_label "h_S3"
 		(shape input)
 		(at 218.44 101.6 180)
@@
 		)
 	)
-	(hierarchical_label "IN_S2"
+	(hierarchical_label "h_S2"
 		(shape input)
 		(at 109.22 99.06 180)
@@
 		)
 	)
-	(hierarchical_label "IN_S2"
+	(hierarchical_label "h_S2"
 		(shape input)
 		(at 163.83 99.06 180)
@@
 		)
 	)
-	(hierarchical_label "IN_S3"
+	(hierarchical_label "h_S3"
 		(shape input)
 		(at 163.83 101.6 180)
@@
 		)
 	)
-	(hierarchical_label "IN_S1"
+	(hierarchical_label "h_S1"
 		(shape input)
 		(at 163.83 96.52 180)
@@
 		)
 	)
-	(hierarchical_label "IN_S0"
+	(hierarchical_label "h_S0"
 		(shape input)
 		(at 163.83 93.98 180)
@@
 		)
 	)
-	(hierarchical_label "IN_S1"
+	(hierarchical_label "h_S1"
 		(shape input)
 		(at 109.22 96.52 180)
@@
 		)
 	)
-	(hierarchical_label "IN_S0"
+	(hierarchical_label "h_S0"
 		(shape input)
 		(at 218.44 93.98 180)
@@
 		)
 	)
-	(hierarchical_label "IN_EN2"
+	(hierarchical_label "h_EN2"
 		(shape input)
 		(at 163.83 111.76 180)
@@
 		)
 	)
-	(hierarchical_label "IN_EN1"
+	(hierarchical_label "h_EN1"
 		(shape input)
 		(at 109.22 111.76 180)
@@
 		)
 	)
-	(hierarchical_label "IN_S3"
+	(hierarchical_label "h_S3"
 		(shape input)
 		(at 109.22 101.6 180)
@@
 		)
 	)
-	(hierarchical_label "IN_S2"
+	(hierarchical_label "h_S2"
 		(shape input)
 		(at 218.44 99.06 180)
@@
 		)
 		(instances
-			(project "Test-Provisioning"
-				(path "/8e8be5f8-638f-4444-a554-6e489d9dce34/5d9b3800-6c59-4395-90ab-0ced0ede5c92"
+			(project "Input-Adapter"
+				(path "/8e8be5f8-638f-4444-a554-6e489d9dce34/c22affd4-39f0-4e4c-b4aa-0abccd112ed3"
 					(reference "#PWR03")
 					(unit 1)
@@
 		)
 		(instances
-			(project "Test-Provisioning"
-				(path "/8e8be5f8-638f-4444-a554-6e489d9dce34/5d9b3800-6c59-4395-90ab-0ced0ede5c92"
+			(project "Input-Adapter"
+				(path "/8e8be5f8-638f-4444-a554-6e489d9dce34/c22affd4-39f0-4e4c-b4aa-0abccd112ed3"
 					(reference "#PWR04")
 					(unit 1)
@@
 		)
 		(instances
-			(project "Test-Provisioning"
-				(path "/8e8be5f8-638f-4444-a554-6e489d9dce34/5d9b3800-6c59-4395-90ab-0ced0ede5c92"
+			(project "Input-Adapter"
+				(path "/8e8be5f8-638f-4444-a554-6e489d9dce34/c22affd4-39f0-4e4c-b4aa-0abccd112ed3"
 					(reference "U6")
 					(unit 1)
@@
 		)
 		(instances
-			(project "Test-Provisioning"
-				(path "/8e8be5f8-638f-4444-a554-6e489d9dce34/5d9b3800-6c59-4395-90ab-0ced0ede5c92"
+			(project "Input-Adapter"
+				(path "/8e8be5f8-638f-4444-a554-6e489d9dce34/c22affd4-39f0-4e4c-b4aa-0abccd112ed3"
 					(reference "U5")
 					(unit 1)
@@
 		)
 		(instances
-			(project "Test-Provisioning"
-				(path "/8e8be5f8-638f-4444-a554-6e489d9dce34/5d9b3800-6c59-4395-90ab-0ced0ede5c92"
+			(project "Input-Adapter"
+				(path "/8e8be5f8-638f-4444-a554-6e489d9dce34/c22affd4-39f0-4e4c-b4aa-0abccd112ed3"
 					(reference "C3")
 					(unit 1)
@@
 		)
 		(instances
-			(project "Test-Provisioning"
-				(path "/8e8be5f8-638f-4444-a554-6e489d9dce34/5d9b3800-6c59-4395-90ab-0ced0ede5c92"
+			(project "Input-Adapter"
+				(path "/8e8be5f8-638f-4444-a554-6e489d9dce34/c22affd4-39f0-4e4c-b4aa-0abccd112ed3"
 					(reference "C2")
 					(unit 1)
@@
 		)
 		(instances
-			(project "Test-Provisioning"
-				(path "/8e8be5f8-638f-4444-a554-6e489d9dce34/5d9b3800-6c59-4395-90ab-0ced0ede5c92"
+			(project "Input-Adapter"
+				(path "/8e8be5f8-638f-4444-a554-6e489d9dce34/c22affd4-39f0-4e4c-b4aa-0abccd112ed3"
 					(reference "U4")
 					(unit 1)
@@
 		)
 		(instances
-			(project "Test-Provisioning"
-				(path "/8e8be5f8-638f-4444-a554-6e489d9dce34/5d9b3800-6c59-4395-90ab-0ced0ede5c92"
+			(project "Input-Adapter"
+				(path "/8e8be5f8-638f-4444-a554-6e489d9dce34/c22affd4-39f0-4e4c-b4aa-0abccd112ed3"
 					(reference "J4")
 					(unit 1)
@@
 		)
 		(instances
-			(project "Test-Provisioning"
-				(path "/8e8be5f8-638f-4444-a554-6e489d9dce34/5d9b3800-6c59-4395-90ab-0ced0ede5c92"
+			(project "Input-Adapter"
+				(path "/8e8be5f8-638f-4444-a554-6e489d9dce34/c22affd4-39f0-4e4c-b4aa-0abccd112ed3"
 					(reference "#PWR07")
 					(unit 1)
@@
 		)
 		(instances
-			(project "Test-Provisioning"
-				(path "/8e8be5f8-638f-4444-a554-6e489d9dce34/5d9b3800-6c59-4395-90ab-0ced0ede5c92"
+			(project "Input-Adapter"
+				(path "/8e8be5f8-638f-4444-a554-6e489d9dce34/c22affd4-39f0-4e4c-b4aa-0abccd112ed3"
 					(reference "#PWR08")
 					(unit 1)
@@
 		)
 		(instances
-			(project "Test-Provisioning"
-				(path "/8e8be5f8-638f-4444-a554-6e489d9dce34/5d9b3800-6c59-4395-90ab-0ced0ede5c92"
+			(project "Input-Adapter"
+				(path "/8e8be5f8-638f-4444-a554-6e489d9dce34/c22affd4-39f0-4e4c-b4aa-0abccd112ed3"
 					(reference "#PWR05")
 					(unit 1)
@@
 		)
 		(instances
-			(project "Test-Provisioning"
-				(path "/8e8be5f8-638f-4444-a554-6e489d9dce34/5d9b3800-6c59-4395-90ab-0ced0ede5c92"
+			(project "Input-Adapter"
+				(path "/8e8be5f8-638f-4444-a554-6e489d9dce34/c22affd4-39f0-4e4c-b4aa-0abccd112ed3"
 					(reference "C1")
 					(unit 1)
@@
 		)
 		(instances
-			(project "Test-Provisioning"
-				(path "/8e8be5f8-638f-4444-a554-6e489d9dce34/5d9b3800-6c59-4395-90ab-0ced0ede5c92"
+			(project "Input-Adapter"
+				(path "/8e8be5f8-638f-4444-a554-6e489d9dce34/c22affd4-39f0-4e4c-b4aa-0abccd112ed3"
 					(reference "J7")
 					(unit 1)
@@
 		)
 		(instances
-			(project "Test-Provisioning"
-				(path "/8e8be5f8-638f-4444-a554-6e489d9dce34/5d9b3800-6c59-4395-90ab-0ced0ede5c92"
+			(project "Input-Adapter"
+				(path "/8e8be5f8-638f-4444-a554-6e489d9dce34/c22affd4-39f0-4e4c-b4aa-0abccd112ed3"
 					(reference "#PWR09")
 					(unit 1)

Commit message: Save agreed Input Adapter reference connector polarity
Parts:
- renumbered J7 to TP1
Connections:
- net MB_3V3_SYS: now also TP1.2 (Pin_2); no longer TP1.1 (Pin_1)
- net MB_GND: now also TP1.1 (Pin_1); no longer TP1.2 (Pin_2)
Changed lines of the file:
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@@
 	)
 	(label "MB_GND"
-		(at 257.81 124.46 90)
+		(at 260.35 124.46 90)
 		(effects
 			(font
@@
 	)
 	(label "MB_3V3_SYS"
-		(at 260.35 124.46 90)
+		(at 257.81 124.46 90)
 		(effects
 			(font
@@
 		(dnp yes)
 		(fields_autoplaced yes)
-		(property "Reference" "J7"
+		(property "Reference" "TP1"
 			(at 261.62 127.6349 90)
 			(show_name no)
@@
 			(project "Input-Adapter"
 				(path "/8e8be5f8-638f-4444-a554-6e489d9dce34/c22affd4-39f0-4e4c-b4aa-0abccd112ed3"
-					(reference "J7")
+					(reference "TP1")
 					(unit 1)
 				)
