File: hardware/kicad/MainBoards/Input-Adapter/Input-Adapter.kicad_pcb (KiCad board)
At the start: 2 copper layers, 35 x 73.7 mm, 9 parts, among them J1 Conn_02x05_Odd_Even, J4 ESP32_DevKitC_TestPlug, J7 Conn_01x02_Socket, U4 CD74HC4067M, U5 CD74HC4067M, U6 CD74HC4067M

Commit message: Save agreed Input Adapter reference connector polarity
Parts:
- moved TP1 2.40 mm to (145.4, 91.6), turned to 180 degrees
- renumbered J7 to TP1
Connections:
- TP1 pad 1: /IN/MB_3V3_SYS -> /IN/MB_GND
- TP1 pad 2: /IN/MB_GND -> /IN/MB_3V3_SYS
Routing:
- net /IN/MB_3V3_SYS: track 10.4 -> 11.2 mm
Other:
- board text added: "3V3"
- board text added: "GND"
Changed lines of the file:
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@@
 	)
 	(footprint "Connector_PinHeader_2.54mm:PinHeader_1x02_P2.54mm_Vertical"
-		(locked yes)
 		(layer "F.Cu")
-		(at 145.41 89.16)
+		(at 145.39 91.56 180)
 		(descr "Through hole straight pin header, 1x02, 2.54mm pitch, single row")
 		(tags "Through hole pin header THT 1x02 2.54mm single row")
-		(property "Reference" "J7"
-			(at 0.05 5.15 0)
+		(property "Reference" "TP1"
+			(at 0.02 -2.75 0)
 			(layer "F.SilkS")
 			(effects
@@
 		(duplicate_pad_numbers_are_jumpers no)
 		(fp_line
-			(start -1.38 -1.38)
-			(end 0 -1.38)
+			(start 1.38 1.27)
+			(end 1.38 3.92)
 			(stroke
 				(width 0.12)
@@
 		)
 		(fp_line
-			(start -1.38 0)
-			(end -1.38 -1.38)
+			(start -1.38 3.92)
+			(end 1.38 3.92)
 			(stroke
 				(width 0.12)
@@
 		(fp_line
 			(start -1.38 1.27)
-			(end -1.38 3.92)
+			(end 1.38 1.27)
 			(stroke
 				(width 0.12)
@@
 		(fp_line
 			(start -1.38 1.27)
-			(end 1.38 1.27)
+			(end -1.38 3.92)
 			(stroke
 				(width 0.12)
@@
 		)
 		(fp_line
-			(start -1.38 3.92)
-			(end 1.38 3.92)
+			(start -1.38 0)
+			(end -1.38 -1.38)
 			(stroke
 				(width 0.12)
@@
 		)
 		(fp_line
-			(start 1.38 1.27)
-			(end 1.38 3.92)
+			(start -1.38 -1.38)
+			(end 0 -1.38)
 			(stroke
 				(width 0.12)
@@
 		)
 		(fp_line
-			(start -1.27 -0.635)
-			(end -0.635 -1.27)
+			(start 1.27 3.81)
+			(end -1.27 3.81)
 			(stroke
 				(width 0.1)
@@
 		)
 		(fp_line
-			(start -1.27 3.81)
-			(end -1.27 -0.635)
+			(start 1.27 -1.27)
+			(end 1.27 3.81)
 			(stroke
 				(width 0.1)
@@
 		)
 		(fp_line
-			(start 1.27 -1.27)
-			(end 1.27 3.81)
+			(start -1.27 3.81)
+			(end -1.27 -0.635)
 			(stroke
 				(width 0.1)
@@
 		)
 		(fp_line
-			(start 1.27 3.81)
-			(end -1.27 3.81)
+			(start -1.27 -0.635)
+			(end -0.635 -1.27)
 			(stroke
 				(width 0.1)
@@
 		)
 		(pad "1" thru_hole rect
-			(at 0 0)
+			(at 0 0 180)
 			(size 1.7 1.7)
 			(drill 1)
 			(layers "*.Cu" "*.Mask")
 			(remove_unused_layers no)
-			(net "/IN/MB_3V3_SYS")
+			(net "/IN/MB_GND")
 			(pinfunction "Pin_1_1")
 			(pintype "passive")
 		)
 		(pad "2" thru_hole circle
-			(at 0 2.54)
+			(at 0 2.54 180)
 			(size 1.7 1.7)
 			(drill 1)
 			(layers "*.Cu" "*.Mask")
 			(remove_unused_layers no)
-			(net "/IN/MB_GND")
+			(net "/IN/MB_3V3_SYS")
 			(pinfunction "Pin_2_2")
 			(pintype "passive")
@@
 		(layer "Edge.Cuts")
 	)
+	(gr_text "GND"
+		(at 147.02 92.14 0)
+		(layer "F.SilkS")
+		(effects
+			(font
+				(size 0.8 0.8)
+				(thickness 0.08)
+			)
+			(justify left bottom)
+		)
+	)
+	(gr_text "3V3"
+		(at 147.09 89.64 0)
+		(layer "F.SilkS")
+		(effects
+			(font
+				(size 0.8 0.8)
+				(thickness 0.08)
+			)
+			(justify left bottom)
+		)
+	)
 	(gr_text "${TITLE}, ${REVISION}"
 		(at 117.68 80.99 90)
@@
 	(segment
 		(start 141.85 84.71)
+		(end 145.39 88.25)
+		(width 0.2)
+		(layer "F.Cu")
+		(net "/IN/MB_3V3_SYS")
+	)
+	(segment
+		(start 145.39 89.02)
+		(end 145.39 88.25)
+		(width 0.2)
+		(layer "F.Cu")
+		(net "/IN/MB_3V3_SYS")
+	)
+	(segment
+		(start 145.39 88.25)
 		(end 145.41 88.27)
 		(width 0.2)
@@
 	)
 	(segment
-		(start 142.554314 85.98)
+		(start 141.82 85.98)
 		(end 137.34 85.98)
 		(width 0.2)
@@
 	)
 	(segment
-		(start 144.26 87.685686)
-		(end 142.554314 85.98)
+		(start 145.41 91.7)
+		(end 142.67 88.96)
 		(width 0.2)
 		(layer "F.Cu")
@@
 	)
 	(segment
-		(start 145.41 91.7)
-		(end 144.26 90.55)
+		(start 142.67 86.83)
+		(end 141.82 85.98)
 		(width 0.2)
 		(layer "F.Cu")
@@
 	)
 	(segment
-		(start 144.26 90.55)
-		(end 144.26 87.685686)
+		(start 142.67 88.96)
+		(end 142.67 86.83)
 		(width 0.2)
 		(layer "F.Cu")
